File: board/t80-psu5.kicad_sch (KiCad schematic)
At the start: 28 parts

Commit message: WIP
Parts:
- removed ? (x2): (no value), symbol Device:C
- removed ?: (no value), symbol Drake:FR8205
- removed ? (x3): (no value), symbol Device:R
- removed ?: (no value), symbol Device:L
- removed ? (x2): (no value), symbol Device:C_Polarized
- removed NT1: NetTie_2, symbol Device:NetTie_2
Connections:
- net +12V is gone; now on net +5V: ?.1, ?.2, ?.2, ?.2 (Pin_2), ?.5 (VIN)

Commit message: WIP
Parts:
- removed ? (x2): (no value), symbol Device:C_Polarized
- removed ?: (no value), symbol Drake:FR8205
- removed ? (x2): (no value), symbol Device:C
- removed ? (x3): (no value), symbol Device:R
- removed ?: (no value), symbol Device:L
- removed NT1 (x4): NetTie_2, symbol Device:NetTie_2
- removed X1 (x2): ~, symbol t80:t80-pin-header
- added C1 (x2): 10u, Capacitor_SMD:C_0805_2012Metric_Pad1.18x1.45mm_HandSolder, symbol Device:C
- added U1: LM1117-3.3, symbol Regulator_Linear:LM1117-3.3
- added X1: ~, symbol t80:t80-pin-header
Connections:
- net +3V3: now also C1.1, U1.2 (VO), X1.4 (3V3); no longer ?.2 (A)
- net +5V: now also ?.2 (A), C1.1, U1.3 (VI), X1.10 (5V)
- net GND: now also C1.2, C1.2, U1.1 (GND), X1.1 (GND), X1.9 (GND)
- no-connect marks 0 -> 4

Commit message: WIP
Connections:
- net +5V: now also X1.8 (5V); no longer X1.10 (5V)
- net GND: now also X1.7 (GND); no longer X1.9 (GND)
Changed lines of the file:
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@@
     )
     (pin "1")
-    (pin "10")
     (pin "2")
     (pin "3")
     (pin "4")
+    (pin "5")
+    (pin "6")
     (pin "7")
     (pin "8")
-    (pin "9")
   )
   (symbol (lib_id "Device:R") (at 87.63 121.92 90) (unit 1)
@@
     )
     (path "/ba2b1566-9a22-409b-9f49-2d8d61922e8f"
-      (reference "X3") (unit 1) (value "~") (footprint "Connector_IDC:IDC-Header_2x05_P2.54mm_Vertical")
+      (reference "X3") (unit 1) (value "~") (footprint "Connector_IDC:IDC-Header_2x04_P2.54mm_Vertical")
     )
   )
